File: Hardware/Sensors_RTC.sch (KiCad schematic (older format))
At the start: 12 parts, among them J1 BME680, U2 DS3231M, U3 Adafruit_BME680

Commit message: [Hardware] Replaced each supply part by a generic one to avoid creating a new symbol for every supply part.
Parts:
- removed U3: Adafruit_BME680, Empty_Footprint:Empty_Footprint, symbol Adafruit_BME680:Adafruit_BME680
Changed lines of the file:
@@
 $Descr A4 11693 8268
 encoding utf-8
-Sheet 2 4
+Sheet 2 5
 Title "Sensors and real-time clock"
 Date ""
@@
 BME680_CS
 $Comp
-L Adafruit_BME680:Adafruit_BME680 U3
-U 1 1 5E7A3D1F
-P 8600 1250
-F 0 "U3" H 9028 1296 50  0000 L CNN
-F 1 "Adafruit_BME680" H 9028 1205 50  0000 L CNN
-F 2 "Empty_Footprint:Empty_Footprint" H 8600 1250 50  0001 C CNN
-F 3 "" H 8600 1250 50  0001 C CNN
-	1    8600 1250
-	1    0    0    -1
-$EndComp
-$Comp
 L Device:Battery BT1
